File: Hardware/Sensoren.sch (KiCad schematic (older format))
At the start: 29 parts, among them J1 CH0, J2 CH1, J3 CH2, J4 CH3, J5 CH4, J6 CH5, P6 SPI_DEBUG, U1 MCP3208

Commit message: fixed all known hardware issues
Parts:
- removed W1, W2, W3, W4, W5, W6: TEST_1P, Measurement_Points:Measurement_Point_Round-SMD-Pad_Small, symbol TEST_1P
- added C10, C11, C12, C13, C14, C9: 10nF, Capacitors_SMD:C_0603, symbol C_Small
- U1: symbol MCP3208 -> MCP3208-RESCUE-Lüftersteuerung
Connections:
- net CH0: now also J1.2, C9.1; no longer J1.1
- net CH1: now also J2.2, C10.1; no longer J2.1
- net CH2: now also J3.2, C11.1; no longer J3.1
- net CH3: now also J4.2, C12.1; no longer J4.1
- net CH4: now also J5.2, C13.1; no longer J5.1
- net CH5: now also J6.2, C14.1; no longer J6.1
- net GND: now also J1.1, J2.1, J3.1, J4.1, J5.1, J6.1, C10.2, C11.2, C12.2, C13.2, C14.2, C9.2; no longer J1.2, J2.2, J3.2, J4.2, J5.2, J6.2
- no-connect marks 0 -> 6
