File: Hardware/mcu.sch (KiCad schematic (older format))
At the start: 26 parts, among them P1 ISP_HEADER, SW1 SW_NB, SW2 SW_INIT, U4 Byteworker, X2 SUB-D9

Commit message: fixed all known hardware issues
Parts:
- D1, D2: footprint SSF_LXH303:SSF-LXH303 -> LEDs:LED_D3.0mm
Changed lines of the file:
@@
 LIBS:Lüftersteuerung
 LIBS:mate-n-lok
-LIBS:mcp3208
 LIBS:tps793
 LIBS:sub-d9
 LIBS:byteworker
 LIBS:mj-2508
+LIBS:mcp3208
 LIBS:Lüftersteuerung-cache
 EELAYER 25 0
@@
 F 0 "D1" H 7250 4525 50  0000 L CNN
 F 1 "Led_Status" H 7125 4300 50  0000 L CNN
-F 2 "SSF_LXH303:SSF-LXH303" V 7300 4400 50  0001 C CNN
+F 2 "LEDs:LED_D3.0mm" V 7300 4400 50  0001 C CNN
 F 3 "" V 7300 4400 50  0000 C CNN
 	1    7300 4400
@@
 F 0 "D2" H 7250 4725 50  0000 L CNN
 F 1 "Led_OK" H 7125 4500 50  0000 L CNN
-F 2 "SSF_LXH303:SSF-LXH303" V 7300 4600 50  0001 C CNN
+F 2 "LEDs:LED_D3.0mm" V 7300 4600 50  0001 C CNN
 F 3 "" V 7300 4600 50  0000 C CNN
 	1    7300 4600
